Commit message: lv2

File: robot_swerve_description/urdf/robot_swerve.urdf (robot description, URDF)
Before this commit: robot robot_swerve, 14 links, 13 joints
Links:
- removed link base_footprint
- removed link hoder_back_left_link_1
- removed link hoder_back_right_link_1
- removed link hoder_front_left_link_1
- removed link hoder_front_right_link_1
- removed link wheel_back_left_link_1
- removed link wheel_back_right_link_1
- added link steering_front_left_link_1, mass 2.725786674997393; collision mesh filename=package://robot_swerve_description/meshes/steering_front_le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 scale=0.001 0.001 0.001; visual mesh filename=package://robot_swerve_description/meshes/steering_front_le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 scale=0.001 0.001 0.001
- added link steering_front_right_link_1, mass 2.7257867924470394; collision mesh filename=package://robot_swerve_description/meshes/steering_front_ri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 scale=0.001 0.001 0.001; visual mesh filename=package://robot_swerve_description/meshes/steering_front_ri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 scale=0.001 0.001 0.001
- added link steering_rear_left_link_1, mass 2.725786615393923; collision mesh filename=package://robot_swerve_description/meshes/steering_rear_lef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 scale=0.001 0.001 0.001; visual mesh filename=package://robot_swerve_description/meshes/steering_rear_lef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 scale=0.001 0.001 0.001
- added link steering_rear_right_link_1, mass 2.7257867677183323; collision mesh filename=package://robot_swerve_description/meshes/steering_rear_rig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 scale=0.001 0.001 0.001; visual mesh filename=package://robot_swerve_description/meshes/steering_rear_rig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 scale=0.001 0.001 0.001
- added link wheel_rear_left_link_1, mass 7.520410979673579; collision mesh filename=package://robot_swerve_description/meshes/wheel_rear_left_l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 scale=0.001 0.001 0.001; visual mesh filename=package://robot_swerve_description/meshes/wheel_rear_left_l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 scale=0.001 0.001 0.001
- added link wheel_rear_right_link_1, mass 7.520363690354945; collision mesh filename=package://robot_swerve_description/meshes/wheel_rear_right_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 scale=0.001 0.001 0.001; visual mesh filename=package://robot_swerve_description/meshes/wheel_rear_right_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 scale=0.001 0.001 0.001
Joints:
- removed joint base_joint
- removed joint hoder_back_left_joint
- removed joint hoder_back_right_joint
- removed joint hoder_front_left_joint
- removed joint hoder_front_right_joint
- removed joint wheel_back_left_joint
- removed joint wheel_back_right_joint
- added joint steering_front_left_joint: type continuous, parent base_link, child steering_front_left_link_1, origin xyz=0.3 0.25 0.15 rpy=0 0 0, axis 0.0 0.0 -1.0, limit lower=-2.1 upper=2.1 effort=5 velocity=6.28
- added joint steering_front_right_joint: type continuous, parent base_link, child steering_front_right_link_1, origin xyz=0.3 -0.25 0.15 rpy=0 0 0, axis 0.0 0.0 -1.0, limit lower=-2.1 upper=2.1 effort=5 velocity=6.28
- added joint steering_rear_left_joint: type continuous, parent base_link, child steering_rear_left_link_1, origin xyz=-0.3 0.25 0.15 rpy=0 0 0, axis 0.0 0.0 -1.0, limit lower=-2.1 upper=2.1 effort=5 velocity=6.28
- added joint steering_rear_right_joint: type continuous, parent base_link, child steering_rear_right_link_1, origin xyz=-0.3 -0.25 0.15 rpy=0 0 0, axis 0.0 0.0 -1.0, limit lower=-2.1 upper=2.1 effort=5 velocity=6.28
- added joint wheel_rear_left_joint: type continuous, parent steering_rear_left_link_1, child wheel_rear_left_link_1, origin xyz=-0.002084 0.0663 -0.139197 rpy=0 0 0, axis 0.0 1.0 0.0, limit effort=1.5 velocity=20
- added joint wheel_rear_right_joint: type continuous, parent steering_rear_right_link_1, child wheel_rear_right_link_1, origin xyz=-0.002085 -0.06638 -0.139197 rpy=0 0 0, axis 0.0 1.0 0.0, limit effort=1.5 velocity=20
- joint wheel_front_left_joint: parent hoder_front_left_link_1 -> steering_front_left_link_1
- joint wheel_front_right_joint: parent hoder_front_right_link_1 -> steering_front_right_link_1

Commit message: lv1

File: robot_swerve_description/urdf/robot_swerve.urdf (robot description, URDF)
Before this commit: robot robot_swerve, 13 links, 12 joints
Joints:
- joint steering_front_left_joint: axis 0.0 0.0 -1.0 -> 0.0 0.0 1.0; limit lower=-2.1 upper=2.1 effort=5 velocity=6.28 -> (none)
- joint steering_front_right_joint: axis 0.0 0.0 -1.0 -> 0.0 0.0 1.0; limit lower=-2.1 upper=2.1 effort=5 velocity=6.28 -> (none)
- joint steering_rear_left_joint: axis 0.0 0.0 -1.0 -> 0.0 0.0 1.0; limit lower=-2.1 upper=2.1 effort=5 velocity=6.28 -> (none)
- joint steering_rear_right_joint: axis 0.0 0.0 -1.0 -> 0.0 0.0 1.0; limit lower=-2.1 upper=2.1 effort=5 velocity=6.28 -> lower=-2.1 upper=2.1 effort=5 velocity=20
- joint wheel_front_left_joint: limit effort=1.5 velocity=20 -> (none)
- joint wheel_front_right_joint: limit effort=1.5 velocity=20 -> (none)
- joint wheel_rear_left_joint: limit effort=1.5 velocity=20 -> (none)
- joint wheel_rear_right_joint: limit effort=1.5 velocity=20 -> (none)
