Commit message: update odom

File: delivery_gazebo/urdf/robot.urdf.xacro (robot description, xacro)
@@ -2,5 +2,6 @@
 <robot xmlns:xacro="http://www.ros.org/wiki/xacro"  name="robot">
     <xacro:include filename="robot_core.xacro"/>
-    <!-- <xacro:include filename="ros2_control.xacro" /> -->
+    <xacro:include filename="materials.xacro"/>
+    <xacro:include filename="robot_control.xacro" />
     <!-- <xacro:include filename="gazebo_control.xacro"/> -->
     <!-- <xacro:include filename="lidar.xacro"/>

File: delivery_gazebo/urdf/robot_core.xacro (robot description, xacro)
@@ -1,17 +1,13 @@
 <?xml version="1.0"?>
 <robot xmlns:xacro="http://www.ros.org/wiki/xacro" >
-    <material name="white">
-        <color rgba="1 1 1 1"/>
-    </material>
-    <material name="black">
-        <color rgba="0 0 0 1"/>
-    </material>
-    <material name="orange">
-        <color rgba="1 0.3 0.1 1"/>
-    </material>
-    <material name="yellow">
-        <color rgba="1 1 0 1"/>
-    </material>
 <link name="base_link">
+</link>
+<!-- BASE_FOOTPRINT LINK -->
+<joint name="base_footprint_joint" type="fixed">
+    <parent link="base_link"/>
+    <child link="base_footprint"/>
+    <origin xyz="0 0 0" rpy="0 0 0"/>
+</joint>
+<link name="base_footprint">
 </link>
 <joint name="chassis_joint" type="fixed">
@@ -33,5 +29,5 @@
       <mesh filename="package://delivery_gazebo/meshes/base_link.stl" scale="0.001 0.001 0.001"/>
     </geometry>
-    <material name="silver"/>
+    <material name="black"/>
   </visual>
   <collision>
@@ -42,4 +38,7 @@
   </collision>
 </link>
+<gazebo reference="chassis">
+        <material>Gazebo/Black</material>
+</gazebo>
 <link name="rl_steer_link_1">
   <inertial>
@@ -53,5 +52,5 @@
       <mesh filename="package://delivery_gazebo/meshes/rl_steer_link_1.stl" scale="0.001 0.001 0.001"/>
     </geometry>
-    <material name="silver"/>
+    <material name="yellow"/>
   </visual>
   <collision>
@@ -62,4 +61,7 @@
   </collision>
 </link>
+<gazebo reference="rl_steer_link_1">
+        <material>Gazebo/Yellow</material>
+</gazebo>
 <link name="rl_wheel_link_1">
   <inertial>
@@ -82,4 +84,8 @@
   </collision>
 </link>
+<gazebo reference="rl_wheel_link_1">
+        <mu1 value="1000000.0"/>
+        <mu2 value="1000000.0"/>
+</gazebo>
 <link name="rr_steer_link_1">
   <inertial>
@@ -93,5 +99,5 @@
       <mesh filename="package://delivery_gazebo/meshes/rr_steer_link_1.stl" scale="0.001 0.001 0.001"/>
     </geometry>
-    <material name="silver"/>
+    <material name="yellow"/>
   </visual>
   <collision>
@@ -102,4 +108,7 @@
   </collision>
 </link>
+<gazebo reference="rr_steer_link_1">
+        <material>Gazebo/Yellow</material>
+</gazebo>
 <link name="rr_wheel_link_1">
   <inertial>
@@ -122,4 +131,8 @@
   </collision>
 </link>
+<gazebo reference="rr_wheel_link_1">
+        <mu1 value="1000000.0"/>
+        <mu2 value="1000000.0"/>
+</gazebo>
 <link name="fr_steer_link_1">
   <inertial>
@@ -133,5 +146,5 @@
       <mesh filename="package://delivery_gazebo/meshes/fr_steer_link_1.stl" scale="0.001 0.001 0.001"/>
     </geometry>
-    <material name="silver"/>
+    <material name="yellow"/>
   </visual>
   <collision>
@@ -142,4 +155,7 @@
   </collision>
 </link>
+<gazebo reference="fr_steer_link_1">
+        <material>Gazebo/Yellow</material>
+</gazebo>
 <link name="fr_wheel_link_1">
   <inertial>
@@ -162,4 +178,8 @@
   </collision>
 </link>
+<gazebo reference="fr_wheel_link_1">
+        <mu1 value="1000000.0"/>
+        <mu2 value="1000000.0"/>
+</gazebo>
 <link name="fl_steer_link_1">
   <inertial>
@@ -173,5 +193,5 @@
       <mesh filename="package://delivery_gazebo/meshes/fl_steer_link_1.stl" scale="0.001 0.001 0.001"/>
     </geometry>
-    <material name="silver"/>
+    <material name="yellow"/>
   </visual>
   <collision>
@@ -182,4 +202,7 @@
   </collision>
 </link>
+<gazebo reference="fl_steer_link_1">
+        <material>Gazebo/Yellow</material>
+</gazebo>
 <link name="fl_wheel_link_1">
   <inertial>
@@ -202,5 +225,9 @@
   </collision>
 </link>
-<joint name="Revolute 1" type="continuous">
+<gazebo reference="fl_wheel_link_1">
+        <mu1 value="1000000.0"/>
+        <mu2 value="1000000.0"/>
+</gazebo>
+<joint name="steering_rear_left_joint" type="continuous">
   <origin xyz="0.3 -0.25 0.15" rpy="0 0 0"/>
   <parent link="chassis"/>
@@ -208,5 +235,5 @@
   <axis xyz="0.0 0.0 -1.0"/>
 </joint>
-<joint name="Revolute 2" type="continuous">
+<joint name="wheel_rear_left_joint" type="continuous">
   <origin xyz="0.026756 -0.061506 -0.139352" rpy="0 0 0"/>
   <parent link="rl_steer_link_1"/>
@@ -214,5 +241,5 @@
   <axis xyz="-0.441333 0.897343 -0.0"/>
 </joint>
-<joint name="Revolute 3" type="continuous">
+<joint name="steering_rear_right_joint" type="continuous">
   <origin xyz="0.3 0.25 0.15" rpy="0 0 0"/>
   <parent link="chassis"/>
@@ -220,5 +247,5 @@
   <axis xyz="0.0 0.0 -1.0"/>
 </joint>
-<joint name="Revolute 4" type="continuous">
+<joint name="wheel_rear_right_joint" type="continuous">
   <origin xyz="0.026756 0.061506 -0.139352" rpy="0 0 0"/>
   <parent link="rr_steer_link_1"/>
@@ -226,5 +253,5 @@
   <axis xyz="-0.441333 -0.897343 -0.0"/>
 </joint>
-<joint name="Revolute 5" type="continuous">
+<joint name="steering_front_right_joint" type="continuous">
   <origin xyz="-0.3 0.25 0.15" rpy="0 0 0"/>
   <parent link="chassis"/>
@@ -232,5 +259,5 @@
   <axis xyz="0.0 0.0 -1.0"/>
 </joint>
-<joint name="Revolute 6" type="continuous">
+<joint name="wheel_front_right_joint" type="continuous">
   <origin xyz="-0.026756 0.061506 -0.139352" rpy="0 0 0"/>
   <parent link="fr_steer_link_1"/>
@@ -238,5 +265,5 @@
   <axis xyz="-0.441333 0.897343 -0.0"/>
 </joint>
-<joint name="Revolute 7" type="continuous">
+<joint name="steering_front_left_joint" type="continuous">
   <origin xyz="-0.3 -0.25 0.15" rpy="0 0 0"/>
   <parent link="chassis"/>
@@ -244,5 +271,5 @@
   <axis xyz="0.0 0.0 -1.0"/>
 </joint>
-<joint name="Revolute 8" type="continuous">
+<joint name="wheel_front_left_joint" type="continuous">
   <origin xyz="-0.026756 -0.061506 -0.139352" rpy="0 0 0"/>
   <parent link="fl_steer_link_1"/>
